File: board/rev2/TouchDRO.brd (EAGLE design)
At the start: 50.8 x 50.8 mm, 29 parts

Commit message: adding latest pcb layout 3d model. finalized rev2 wiring, specifically wider routes on GND and VCC
Connections:
- net +5V: now also VREG33.IN
- net D1: no longer VREG33.IN
Routing:
- net D1: track 27.9 -> 11.7 mm
- net +5V: track 28.1 -> 35.6 mm
- net GND: track 186.6 -> 183.4 mm
- net +3V3: track 84.8 -> 83.0 mm
